File: c3rl-at-r-beta-2.kicad_pcb (KiCad board)
At the start: 2 copper layers, 50 x 50 mm, 113 parts, among them IC1 W25Q16JVUXIQ_TR-W25Q16JVUXIQ_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, J1 USB4105-GF-A-USB4105-GF-A, J2 Conn_01x04_Male_JST_ZE, J3 Conn_01x04_Male_JST_ZE, J4 Conn_01x06_Male_JST_ZE, J5 Conn_01x02_Male_JST, J6 U.FL-R-SMT(01), J7 TFP09-2-12B, J8 SM04B-SRSS-TB(LF)(SN), J9 Conn_01x04_Male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

Commit message: rev 1
Parts:
- removed PS1: AP3418KTR-G1, Libraries:SOT95P282X145-5N
- removed Q6: BC817, Package_TO_SOT_SMD:SOT-23
- removed Q7: AO3401A, Package_TO_SOT_SMD:SOT-23
- removed R21, R30: R_0402, Resistor_SMD:R_0402_1005Metric
- removed R43: R, Resistor_SMD:R_0805_2012Metric
- removed the REF** at (76.0, 122.0)
- added C21: 22u, Capacitor_SMD:C_0603_1608Metric, F.Cu at (84.8, 107.8)
- added C33: 22u, Capacitor_SMD:C_0603_1608Metric, F.Cu at (82.0, 100.2)
- added C34: 22u, Capacitor_SMD:C_0603_1608Metric, F.Cu at (82.0, 98.5)
- added C35: C_0603, Capacitor_SMD:C_0402_1005Metric, F.Cu at (84.5, 95.7)
- added C36: C_0603, Capacitor_SMD:C_0402_1005Metric, F.Cu at (85.5, 95.7)
- added C37: C_0402, Capacitor_SMD:C_0402_1005Metric, F.Cu at (95.5, 92.4)
- added C38: C_0603, Capacitor_SMD:C_0603_1608Metric, F.Cu at (95.2, 93.7)
- added C39: C_0603, Capacitor_SMD:C_0603_1608Metric, F.Cu at (95.2, 85.8)
- added C40: C_0402, Capacitor_SMD:C_0402_1005Metric, F.Cu at (95.5, 87.1)
- added D3: MM5Zxx, Diode_SMD:D_SOD-523, F.Cu at (81.8, 96.0)
- added D4: MM5Zxx, Diode_SMD:D_SOD-523, F.Cu at (90.7, 98.9)
- added J10: Conn_01x02_Male, Connector_JST:JST_PH_S2B-PH-SM4-TB_1x02-1MP_P2.00mm_Horizontal, F.Cu at (77.7, 119.9)
- added J11: Conn_01x02_Male, Connector_PinHeader_2.00mm:PinHeader_1x02_P2.00mm_Vertical, F.Cu at (87.6, 98.2)
- added R44: R_0402, Resistor_SMD:R_0402_1005Metric, F.Cu at (85.5, 98.3)
- added REF**: MountingHole_2.7mm_M2.5_ISO14580, MountingHole:MountingHole_2.7mm_M2.5_ISO14580, F.Cu at (76.0, 101.8)
- added REF**: MountingHole_2.7mm_M2.5_ISO14580, MountingHole:MountingHole_2.7mm_M2.5_ISO14580, F.Cu at (92.5, 78.0)
- added U6: AP62300TWU-7, Libraries:SOT95P280X100-6N, F.Cu at (87.1, 104.5)
- C11: value C_0402 -> C_0603; footprint Capacitor_SMD:C_0402_1005Metric -> Capacitor_SMD:C_0603_1608Metric
- C2, C3: footprint Capacitor_SMD:C_0603_1608Metric -> Capacitor_SMD:C_0402_1005Metric
- C31, C32: value C_0805 -> 22u; footprint Capacitor_SMD:C_0805_2012Metric -> Capacitor_SMD:C_0603_1608Metric
- J5: value Conn_01x02_Male_JST -> Conn_01x02_Male; footprint Connector_JST:JST_XH_B2B-XH-A_1x02_P2.50mm_Vertical -> Connector_PinHeader_1.27mm:PinHeader_1x02_P1.27mm_Vertical
- R29: value R_0402 -> R
- U4: value ATECC608A-SSHDA -> AP2171W; footprint Package_SO:SOIC-8_3.9x4.9mm_P1.27mm -> Package_TO_SOT_SMD:SOT-23-5
- moved G*** 20.1 mm to (98.9, 93.3)
- moved J5 17.6 mm to (79.4, 91.0), turned to 0 degrees
- moved C11 17.5 mm to (83.2, 96.2), turned to 90 degrees
- moved C32 5.55 mm to (87.8, 101.9), turned to 180 degrees
- moved U4 5.15 mm to (95.0, 89.8), turned to -90 degrees
- moved C16 4.64 mm to (99.1, 90.9), turned to -90 degrees
- moved C3 3.80 mm to (90.6, 95.1), turned to 0 degrees
- moved U5 3.58 mm to (99.8, 94.0)
- moved C31 3.47 mm to (86.3, 107.8), turned to 90 degrees
- moved R2 3.40 mm to (80.0, 100.2), turned to 90 degrees
- moved Q1 3.01 mm to (78.3, 97.5)
- moved L2 2.49 mm to (83.2, 103.0), turned to 90 degrees
- moved L1 2.02 mm to (85.5, 80.8)
- moved C27 2.01 mm to (84.0, 80.3)
- moved C26 2.00 mm to (87.0, 80.3)
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Connections:
- net /RP_USB_DM renamed /RP_USB_DN
- C11 pad 1: +3V3 -> /LC_V_BCKP
- C32 pad 1: +3V3 -> Net-(C32-Pad1)
- C32 pad 2: GND -> Net-(C32-Pad2)
- J1 pad S1: Net-(J1-PadS1) -> GND
- J1 pad S2: Net-(J1-PadS1) -> GND
- J1 pad S3: Net-(J1-PadS1) -> GND
- J1 pad S4: Net-(J1-PadS1) -> GND
- J5 pad 1: /VIN -> /LC_RX
- J5 pad 2: GND -> /LC_TX
- L2 pad 1: +3V3 -> Net-(C32-Pad2)
- L2 pad 2: Net-(L2-Pad2) -> +3V3
- R29 pad 1: Net-(Q6-Pad1) -> +3V3
- R29 pad 2: /RP_SENSOR_VDD_1_EN -> /VDD_APDS
- R37 pad 1: Net-(PS1-Pad5) -> +3V3
- R37 pad 2: +3V3 -> Net-(R37-Pad2)
- R38 pad 1: GND -> Net-(R37-Pad2)
- R38 pad 2: Net-(PS1-Pad5) -> GND
- U1 pad 6: unconnected-(U1-Pad6) -> /LC_V_BCKP
- U4 pad 1: (no net) -> /VDD_APDS
- U4 pad 2: (no net) -> GND
- U4 pad 3: (no net) -> unconnected-(U4-Pad3)
- U4 pad 4: GND -> /RP_SENSOR_VDD_1_EN
- U4 pad 5: /I2C_SDA -> +3V3
Routing:
- net /LC_V_BCKP: track 0.00 -> 11.5 mm
- net /I2C_SCL: track 128.5 -> 117.1 mm, vias 11 -> 9
- net /I2C_SDA: track 128.0 -> 118.4 mm
- net /LC_RX: track 0.00 -> 6.70 mm
- net /LC_TX: track 0.00 -> 5.43 mm
- net /VIN: track 11.9 -> 17.1 mm, vias 4 -> 7
- net Net-(Q6-Pad1): track 4.53 -> 0.00 mm
- net +3V3: track 260.3 -> 256.5 mm
- net /LC_RF: track 5.77 -> 2.25 mm
- net Net-(Q6-Pad3): track 3.52 -> 0.00 mm
- net Net-(R37-Pad2): track 0.00 -> 2.56 mm
- net Net-(PS1-Pad5): track 2.39 -> 0.00 mm
- net /LC_RF_IN: track 3.97 -> 5.97 mm
- net Net-(D2-Pad1): track 2.78 -> 4.64 mm
- net /RP_RUN: track 8.01 -> 6.16 mm
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- added copper zone on F.Cu, net Net-(C32-Pad1)
- added copper zone on F.Cu, net Net-(C32-Pad2)
- removed copper zone on F.Cu, net Net-(L2-Pad2)
Other:
- outline, holes or cut-outs redrawn
- board text added: "ATNode-R 2023 c3rl Rev 1"
- board text removed: "ATNode-R 2022 c3rl IN"
