File: c3rl-at-r-beta-2.kicad_sch (KiCad schematic)
At the start: 109 parts, among them IC1 W25Q16JVUXIQ_TR-W25Q16JVUXIQ_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, J1 USB4105-GF-A-USB4105-GF-A, J2 Conn_01x04_Male_JST_ZE, J3 Conn_01x04_Male_JST_ZE, J4 Conn_01x06_Male_JST_ZE, J5 Conn_01x02_Male_JST, J6 U.FL-R-SMT(01), J7 TFP09-2-12B, J8 SM04B-SRSS-TB(LF)(SN), J9 Conn_01x04_Male, Q1 BC817, Q2 BC817, Q3 BSS138, Q4 BSS138, Q5 BC817, Q6 BC817, Q7 AO3401A, SW1 SW_Push_3x4x2_tactile-Switch, SW2 SW_Push_3x4x2_tactile-Switch, SW3 SW_Push_3x4x2_tactile-Switch, U1 LC76F, U2 W25Q32JVSS, U3 RP2040, U4 ATECC608A-SSHDA, U5 ATECC608A-MAHDA, U7 APDS-9306-065, U8 LSM6DSOX, U9 HDC2021DEBT, Y1 ABM8-24.000MHZ-B2-T-ABM8-24.0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

Commit message: rev 1
Parts:
- removed C11: C_0402, Capacitor_SMD:C_0402_1005Metric, symbol c3rl-cnode-beta-1-rescue:C_0402-c3rl
- removed C31, C32: C_0805, Capacitor_SMD:C_0805_2012Metric, symbol c3rl-cnode-beta-1-rescue:C_0805-Device
- removed J5: Conn_01x02_Male_JST, Connector_JST:JST_XH_B2B-XH-A_1x02_P2.50mm_Vertical, symbol c3rl:Conn_01x02_Male_JST
- removed PS1: AP3418KTR-G1, SOT95P282X145-5N, symbol c3rl-cnode-beta-1-rescue:AP3418KTR-G1-AP3418KTR-G1
- removed Q6: BC817, Package_TO_SOT_SMD:SOT-23, symbol Transistor_BJT:BC817
- removed Q7: AO3401A, Package_TO_SOT_SMD:SOT-23, symbol Transistor_FET:AO3401A
- removed R21: R_0402, Resistor_SMD:R_0402_1005Metric, symbol c3rl-cnode-beta-1-rescue:R_0402-c3rl
- removed R29, R30: R_0402, Resistor_SMD:R_0402_1005Metric, symbol c3rl:R_0402
- removed R?: R, Resistor_SMD:R_0805_2012Metric, symbol Device:R
- removed U4: ATECC608A-SSHDA, Package_SO:SOIC-8_3.9x4.9mm_P1.27mm, symbol Security:ATECC608A-SSHDA
- added C11, C38, C39: C_0603, Capacitor_SMD:C_0603_1608Metric, symbol c3rl:C_0603
- added C21, C31, C32, C33, C34: 22u, Capacitor_SMD:C_0603_1608Metric, symbol Device:C
- added C35, C36: C_0603, Capacitor_SMD:C_0402_1005Metric, symbol c3rl:C_0603
- added C37, C40: C_0402, Capacitor_SMD:C_0402_1005Metric, symbol c3rl-cnode-beta-1-rescue:C_0402-c3rl
- added D3, D4: MM5Zxx, Diode_SMD:D_SOD-523, symbol Diode:MM5Zxx
- added J10: Conn_01x02_Male, Connector_JST:JST_PH_S2B-PH-SM4-TB_1x02-1MP_P2.00mm_Horizontal, symbol Connector:Conn_01x02_Male
- added J11: Conn_01x02_Male, Connector_PinHeader_2.00mm:PinHeader_1x02_P2.00mm_Vertical, symbol Connector:Conn_01x02_Male
- added J5: Conn_01x02_Male, Connector_PinHeader_1.27mm:PinHeader_1x02_P1.27mm_Vertical, symbol Connector:Conn_01x02_Male
- added R29: R, Resistor_SMD:R_0402_1005Metric, symbol Device:R
- added R44: R_0402, Resistor_SMD:R_0402_1005Metric, symbol c3rl-cnode-beta-1-rescue:R_0402-c3rl
- added U4: AP2171W, Package_TO_SOT_SMD:SOT-23-5, symbol Power_Management:AP2171W
- added U6: AP62300TWU-7, SOT95P280X100-6N, symbol c3rl-cnode-beta-1-rescue:AP62300TWU-7-AP62300TWU-7
- C2, C3: footprint Capacitor_SMD:C_0603_1608Metric -> Capacitor_SMD:C_0402_1005Metric
- gave numbers to parts that had none: 1
Connections:
- net +3V3: now also L2.2, R37.1, C33.1, C34.1, C37.1, C38.2, D4.1 (K), R29.1, R44.2, U4.5 (IN); no longer L2.1, R37.2
- net GND: now also J1.S1 (SHELL_GND), J1.S2 (SHELL_GND), J1.S3 (SHELL_GND), J1.S4 (SHELL_GND), R38.2, C11.2, C21.1, C31.1, C33.2, C34.2, C35.2, C36.2, C37.2, C38.1, C39.1, C40.2, D3.2 (A), D4.2 (A), J10.2 (Pin_2), J11.1 (Pin_1), U4.2 (GND), U6.1 (GND); no longer R38.1
- net LC_RX: now also J5.1 (Pin_1)
- net LC_TX: now also J5.2 (Pin_2)
- net RP_SENSOR_VDD_1_EN: now also U4.4 (EN)
- net VDD_APDS: now also C39.2, C40.1, R29.2, U4.1 (OUT)
- net VIN: now also C21.2, C31.2, J10.1 (Pin_1), U6.3 (VIN), U6.5 (EN)
- net LC_V_BCKP: now reaches U1.6 (V_BCKP)
- net LC_V_BCKP: now also C11.1, C35.1, C36.1, D3.1 (K), J11.2 (Pin_2), R44.1
- net RP_USB_DM renamed RP_USB_DN
- new net: C32.1, U6.6 (BST)
- new net: C32.2, L2.1, U6.2 (SW)
- new net: R37.2, R38.1, U6.4 (FB)
